File: MCU_board/Router_MCU.kicad_pcb (KiCad board)
At the start: 2 copper layers, 157.6 x 116.2 mm, 72 parts, among them J1 Header, T1 HY601742, U1 MYC-YT507H, U2 TPS54540, U3 LAN8720A, X1 S4B-XH, X2 S4B-XH, X3 S4B-XH, X4 S4B-XH, X5 B2B-XH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

Commit message: routing procs
Parts:
- removed H6: M3, MountingHole:MountingHole_3.5mm_Pad
- X1, X2, X3, X4: value S4B-XH -> B4B-XH; footprint Connector_JST:JST_XH_S4B-XH-A_1x04_P2.50mm_Horizontal -> Connector_JST:JST_XH_B4B-XH-A_1x04_P2.50mm_Vertical
- moved H1 149.3 mm to (116.3, 76.8)
- moved R25 138.6 mm to (162.2, 162.4)
- moved H3 117.2 mm to (116.3, 146.8)
- moved C8 102.7 mm to (164.9, 162.4)
- moved R3 99.8 mm to (181.3, 68.4)
- moved R4 98.2 mm to (180.9, 63.5)
- moved H5 95.3 mm to (161.3, 76.8)
- moved H4 74.7 mm to (206.3, 146.8)
- moved J1 69.7 mm to (190.0, 63.6)
- moved X6 68.8 mm to (173.0, 154.9), turned to 90 degrees
- moved H2 57.9 mm to (206.3, 76.8)
- moved X5 54.3 mm to (197.4, 66.2)
- moved R21 53.0 mm to (265.5, 140.7)
- moved R12 46.3 mm to (265.8, 137.7)
- moved U1 44.5 mm to (147.8, 110.9), turned to -90 degrees
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Other:
- board size 157.6 x 116.2 mm -> 99 x 84 mm

Commit message: Modems board ready
Parts:
- added C23: 100u 50V, Capacitor_SMD:CP_Elec_10x10.5, F.Cu at (224.6, 78.5)
Changed lines of the file:
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@@
+    )
+  )
+  (footprint "Capacitor_SMD:CP_Elec_10x10.5" (layer "F.Cu")
+    (at 224.6 78.55)
+    (descr "SMD capacitor, aluminum electrolytic, Vishay 1010, 10.0x10.5mm, http://www.vishay.com/docs/28395/150crz.pdf")
+    (tags "capacitor electrolytic")
+    (property "Sheetfile" "Router_MCU.kicad_sch")
+    (property "Sheetname" "")
+    (attr smd)
+    (fp_text reference "C23" (at 0 -6.3) (layer "F.SilkS")
+      (effects (font (size 1 1) (thickness 0.15)))
+    )
+    (fp_text value "100u 50V" (at 0 6.3) (layer "F.Fab")
+      (effects (font (size 1 1) (thickness 0.15)))
+    )
+    (fp_text user "${REFERENCE}" (at 0 0) (layer "F.Fab")
+      (effects (font (size 1 1) (thickness 0.15)))
+    )
+    (fp_line (start -5.36 -4.295563) (end -5.36 -1.51) (layer "F.SilkS") (width 0.12))
+    (fp_line (start -5.36 4.295563) (end -4.295563 5.36) (layer "F.SilkS") (width 0.12))
+    (fp_line (start -5.36 4.295563) (end -5.36 1.51) (layer "F.SilkS") (width 0.12))
+    (fp_line (start -6.85 -2.76) (end -5.6 -2.76) (layer "F.SilkS") (width 0.12))
+    (fp_line (start -4.295563 5.36) (end 5.36 5.36) (layer "F.SilkS") (width 0.12))
+    (fp_line (start 5.36 -5.36) (end 5.36 -1.51) (layer "F.SilkS") (width 0.12))
+    (fp_line (start -4.295563 -5.36) (end 5.36 -5.36) (layer "F.SilkS") (width 0.12))
+    (fp_line (start -5.36 -4.295563) (end -4.295563 -5.36) (layer "F.SilkS") (width 0.12))
+    (fp_line (start -6.225 -3.385) (end -6.225 -2.135) (layer "F.SilkS") (width 0.12))
+    (fp_line (start 5.36 5.36) (end 5.36 1.51) (layer "F.SilkS") (width 0.12))
+    (fp_line (start -5.5 -4.35) (end -4.35 -5.5) (layer "F.CrtYd") (width 0.05))
+    (fp_line (start -6.65 1.5) (end -5.5 1.5) (layer "F.CrtYd") (width 0.05))
+    (fp_line (start -5.5 4.35) (end -4.35 5.5) (layer "F.CrtYd") (width 0.05))
+    (fp_line (start 6.65 1.5) (end 5.5 1.5) (layer "F.CrtYd") (width 0.05))
+    (fp_line (start -5.5 -1.5) (end -6.65 -1.5) (layer "F.CrtYd") (width 0.05))
+    (fp_line (start 6.65 -1.5) (end 6.65 1.5) (layer "F.CrtYd") (width 0.05))
+    (fp_line (start 5.5 -1.5) (end 6.65 -1.5) (layer "F.CrtYd") (width 0.05))
+    (fp_line (start -4.35 5.5) (end 5.5 5.5) (layer "F.CrtYd") (width 0.05))
+    (fp_line (start 5.5 1.5) (end 5.5 5.5) (layer "F.CrtYd") (width 0.05))
+    (fp_line (start -4.35 -5.5) (end 5.5 -5.5) (layer "F.CrtYd") (width 0.05))
+    (fp_line (start -5.5 1.5) (end -5.5 4.35) (layer "F.CrtYd") (width 0.05))
+    (fp_line (start -5.5 -4.35) (end -5.5 -1.5) (layer "F.CrtYd") (width 0.05))
+    (fp_line (start 5.5 -5.5) (end 5.5 -1.5) (layer "F.CrtYd") (width 0.05))
+    (fp_line (start -6.65 -1.5) (end -6.65 1.5) (layer "F.CrtYd") (width 0.05))
+    (fp_line (start -5.25 -4.25) (end -5.25 4.25) (layer "F.Fab") (width 0.1))
+    (fp_line (start -4.558325 -1.7) (end -3.558325 -1.7) (layer "F.Fab") (width 0.1))
+    (fp_line (start -5.25 4.25) (end -4.25 5.25) (layer "F.Fab") (width 0.1))
+    (fp_line (start -4.25 5.25) (end 5.25 5.25) (layer "F.Fab") (width 0.1))
+    (fp_line (start 5.25 -5.25) (end 5.25 5.25) (layer "F.Fab") (width 0.1))
+    (fp_line (start -4.058325 -2.2) (end -4.058325 -1.2) (layer "F.Fab") (width 0.1))
+    (fp_line (start -4.25 -5.25) (end 5.25 -5.25) (layer "F.Fab") (width 0.1))
+    (fp_line (start -5.25 -4.25) (end -4.25 -5.25) (layer "F.Fab") (width 0.1))
+    (fp_circle (center 0 0) (end 5 0) (layer "F.Fab") (width 0.1) (fill none))
+    (pad "1" smd roundrect (at -4.2 0) (size 4.4 2.5) (layers "F.Cu" "F.Paste" "F.Mask") (roundrect_rratio 0.1)
+      (net 5 "Net-(C5-Pad1)") (pintype "passive"))
+    (pad "2" smd roundrect (at 4.2 0) (size 4.4 2.5) (layers "F.Cu" "F.Paste" "F.Mask") (roundrect_rratio 0.1)
+      (net 2 "GND") (pintype "passive"))
+    (model "${KICAD6_3DMODEL_DIR}/Capacitor_SMD.3dshapes/CP_Elec_10x10.5.wrl"
+      (offset (xyz 0 0 0))
+      (scale (xyz 1 1 1))
+      (rotate (xyz 0 0 0))
     )
   )

Commit message: mcu_pdb_routing
Parts:
- moved R12 181.7 mm to (86.5, 108.8)
- moved C12 154.3 mm to (100.2, 110.3)
- moved C14 153.9 mm to (98.6, 112.2)
- moved C19 152.7 mm to (104.7, 96.5)
- moved D4 149.7 mm to (99.9, 103.6)
- moved R15 148.5 mm to (96.9, 110.2)
- moved C7 146.4 mm to (90.7, 113.2)
- moved C5 146.0 mm to (90.6, 110.2)
- moved U2 140.2 mm to (91.9, 104.7)
- moved C21 139.7 mm to (104.7, 94.0)
- moved R20 137.8 mm to (109.4, 108.0)
- moved C18 137.7 mm to (104.8, 99.1)
- moved R19 137.5 mm to (106.0, 108.0)
- moved C15 134.3 mm to (97.6, 106.8)
- moved C2 128.9 mm to (169.7, 82.3)
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Routing:
- net Net-(C16-Pad1): track 0.00 -> 44.7 mm
- net /USB0_N: track 0.00 -> 40.7 mm
- net /USB0_P: track 0.00 -> 39.7 mm
- net /USB1_N: track 0.00 -> 39.2 mm
- net /USB1_P: track 0.00 -> 38.3 mm
- net /TXD1: track 0.00 -> 38.0 mm, vias 0 -> 2
- net /PHY_RST: track 0.00 -> 36.6 mm, vias 0 -> 2
- net /TXD0: track 0.00 -> 36.4 mm, vias 0 -> 2
- net /MDC: track 0.00 -> 34.5 mm, vias 0 -> 2
- net /MDIO: track 0.00 -> 32.6 mm, vias 0 -> 2
- net /SD0_D2: track 0.00 -> 32.4 mm
- net /SD0_D3: track 0.00 -> 32.2 mm
- net /RXD1: track 0.00 -> 30.1 mm, vias 0 -> 2
- net /RXD0: track 0.00 -> 29.8 mm, vias 0 -> 2
- net /USB3_N: track 0.00 -> 28.9 mm
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
Commit message: mcu_pdb_routing
Parts:
- moved X5 81.9 mm to (206.5, 129.4), turned to -90 degrees
- moved C23 67.2 mm to (120.6, 87.2), turned to 180 degrees
- moved C7 61.1 mm to (137.7, 74.1)
- moved C5 57.8 mm to (137.7, 76.5)
- moved L1 57.2 mm to (149.5, 83.2)
- moved C18 55.9 mm to (155.4, 75.3), turned to 90 degrees
- moved R12 54.1 mm to (131.9, 79.4), turned to -90 degrees
- moved C19 52.6 mm to (152.8, 75.4), turned to 90 degrees
- moved U2 49.4 mm to (135.6, 81.7), turned to -90 degrees
- moved C21 49.3 mm to (150.3, 75.4), turned to 90 degrees
- moved D4 45.3 mm to (140.3, 83.1), turned to 90 degrees
- moved C15 44.6 mm to (137.6, 87.1), turned to 90 degrees
- moved R15 44.0 mm to (134.4, 87.1), turned to -90 degrees
- moved C12 42.7 mm to (136.0, 87.1), turned to 90 degrees
- moved C14 42.4 mm to (132.8, 87.1), turned to 90 degrees
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Connections:
- R3 pad 2: /UART0_TX -> /UART0_RX
- R4 pad 2: /UART0_RX -> /UART0_TX
- U1 pad 13: unconnected-(U1-Pad13) -> /M3_ONOFF
- U1 pad 14: unconnected-(U1-Pad14) -> /M2_ONOFF
- U1 pad 16: unconnected-(U1-Pad16) -> /M1_ONOFF
- U1 pad 17: unconnected-(U1-Pad17) -> /M0_ONOFF
- U1 pad 56: /STAT_LED -> unconnected-(U1-Pad56)
- U1 pad 58: /M0_ONOFF -> unconnected-(U1-Pad58)
- U1 pad 59: /M1_ONOFF -> unconnected-(U1-Pad59)
- U1 pad 61: /M2_ONOFF -> unconnected-(U1-Pad61)
- U1 pad 62: /M3_ONOFF -> unconnected-(U1-Pad62)
- U1 pad L2: unconnected-(U1-PadL2) -> /STAT_LED
Routing:
- net Net-(C23-Pad1): track 0.00 -> 178.8 mm
- net /M0_ONOFF: track 0.00 -> 75.8 mm, vias 0 -> 2
- net /M1_ONOFF: track 0.00 -> 63.9 mm, vias 0 -> 2
- net /M2_ONOFF: track 0.00 -> 62.0 mm, vias 0 -> 2
- net /M3_ONOFF: track 0.00 -> 54.4 mm, vias 0 -> 2
- net GND: track 7.85 -> 56.7 mm, vias 12 -> 74
- net /STAT_LED: track 0.00 -> 37.3 mm, vias 0 -> 1
- net /VIN1: track 0.00 -> 34.4 mm
- net /UART0_RX: track 0.00 -> 31.1 mm, vias 0 -> 1
- net +5V: track 0.00 -> 30.9 mm, vias 0 -> 2
- net /VIN2: track 0.00 -> 29.9 mm
- net /UART0_TX: track 0.00 -> 27.4 mm, vias 0 -> 1
- net /SD0_D0: track 27.4 -> 46.3 mm, vias 1 -> 0
- net /SD0_D1: track 27.7 -> 45.9 mm
- net /SD0_CMD: track 28.5 -> 46.5 mm
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- added copper zone on B.Cu, net +3V3
- added copper zone on F.Cu, net +3V3
- added copper zone on F.Cu, net +5V
- added copper zone on B.Cu, net GND
- added copper zone on F.Cu, net GND
- added copper zone on F.Cu, net Net-(C15-Pad2)
Other:
- board size 99 x 84 mm -> 99 x 84.5 mm
- board text added: "RX TX GND"

Commit message: Ready for order
Routing:
- net GND: vias 74 -> 223

Commit message: remove modems gpio ctrls
Parts:
- R13, R14: value 75 -> 75R
- U2: value TPS54540 -> TPS54340
Connections:
- U1 pad 13: /M3_ONOFF -> unconnected-(U1-Pad13)
- U1 pad 14: /M2_ONOFF -> unconnected-(U1-Pad14)
- U1 pad 16: /M1_ONOFF -> unconnected-(U1-Pad16)
- U1 pad 17: /M0_ONOFF -> unconnected-(U1-Pad17)
- X1 pad 1: /M0_ONOFF -> GND
- X2 pad 1: /M1_ONOFF -> GND
- X3 pad 1: /M2_ONOFF -> GND
- X4 pad 1: /M3_ONOFF -> GND
Routing:
- net /M0_ONOFF: track 75.8 -> 0.00 mm, vias 2 -> 0
- net /M1_ONOFF: track 63.9 -> 0.00 mm, vias 2 -> 0
- net /M2_ONOFF: track 62.0 -> 0.00 mm, vias 2 -> 0
- net /M3_ONOFF: track 54.4 -> 0.00 mm, vias 2 -> 0
