File: MCU_board/Router_MCU.kicad_sch (KiCad schematic)
At the start: 61 parts

Commit message: routing procs
Parts:
- removed C?: 0.1u, Capacitor_SMD:C_0603_1608Metric, symbol Device:C
- removed D?: 2A, symbol Device:D_Bridge_+AA-
- removed R? (x2): 470R, Resistor_SMD:R_0603_1608Metric, symbol Device:R
- removed X?: HR911105A, oca_proj:HANRUN_HR911105A, symbol HR911105A:HR911105A
- removed X?: Conn_01x02, symbol Connector_Generic:Conn_01x02
- added C10: 1n 2kV, Capacitor_SMD:C_1206_3216Metric, symbol Device:C
- added C6: 0.1u, Capacitor_SMD:C_0603_1608Metric, symbol Device:C
- added D1: DB107S, Diode_SMD:Diode_Bridge_OnSemi_SDIP-4L, symbol Device:D_Bridge_+-AA
- added D2: TVS, Diode_SMD:D_SMA, symbol Device:D_Zener
- added H1, H2, H3, H4, H5, H6: M3, MountingHole:MountingHole_3.5mm_Pad, symbol Mechanical:MountingHole_Pad
- added R13, R14: 75, Resistor_SMD:R_0603_1608Metric, symbol Device:R
- added R23, R24: 470R, Resistor_SMD:R_0603_1608Metric, symbol Device:R
- added T1: HY601742, Transformer_SMD:Transformer_Ethernet_Bourns_PT61017PEL, symbol Transformer:PT61017PEL
- added X5: B2B-XH, Connector_JST:JST_XH_B2B-XH-A_1x02_P2.50mm_Vertical, symbol Connector_Generic:Conn_01x02
- added X7: RJ45, Connector_RJ:RJ45_Amphenol_RJHSE538X, symbol Connector:RJ45_LED_Shielded
- C1: renamed from C?; footprint (none) -> Capacitor_SMD:C_0805_2012Metric
- C18, C19, C21, C5, C7: renamed from C?; footprint (none) -> Capacitor_SMD:C_1206_3216Metric
- C2, C8: renamed from C?; footprint (none) -> Capacitor_SMD:C_0603_1608Metric
- D3: renamed from D?; footprint (none) -> LED_THT:LED_D3.0mm
- D4: renamed from D?; value SS310 -> SS540
- J1: renamed from J?; footprint (none) -> Connector_PinHeader_2.54mm:PinHeader_1x03_P2.54mm_Vertical
- L1: renamed from L?; footprint Inductor_SMD:L_Abracon_ASPI-0630LR -> Inductor_SMD:L_Sunlord_MWSA1004S
- R2, R3, R4: renamed from R?; footprint (none) -> Resistor_SMD:R_0603_1608Metric
- U1: renamed from U?; footprint (none) -> MYC-Y6UL:MYC-YT507H
- X1, X2, X3, X4: renamed from X?; value B4B-XH -> S4B-XH; footprint (none) -> Connector_JST:JST_XH_S4B-XH-A_1x04_P2.50mm_Horizontal
- X6: renamed from X?; footprint TFP09212B -> proj:TFP09212B
- Y1: renamed from Y?; footprint (none) -> Oscillator:Oscillator_SMD_Abracon_ASE-4Pin_3.2x2.5mm
- gave numbers to parts that had none: 33
Connections:
- net ETH_LED1: now also R24.2
- net ETH_LED2: now also R23.2
- net GND: now also C10.1, C6.2, D1.2 (-), D2.2 (A), H1.1, H2.1, H3.1, H4.1, H5.1, H6.1, X5.2 (Pin_2), X7.11, X7.9, X7.SH
- net RXN: now also T1.3 (TD-)
- net RXP: now also T1.1 (TD+)
- net TXN: now also T1.8 (RD-)
- net TXP: now also T1.6 (RD+)
- net at C16.1, C17.1, FB1.2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: now also C6.1, T1.2 (C_TD), T1.7 (C_RD)
- net M0_ONOFF: now reaches U1.58 (NCSI0-D14)
- net M0_ONOFF: now also X1.1 (Pin_1)
- net M1_ONOFF: now reaches U1.59 (NCSI0-D13)
- net M1_ONOFF: now also X2.1 (Pin_1)
- net M2_ONOFF: now reaches U1.61 (NCSI0-D12)
- net M2_ONOFF: now also X3.1 (Pin_1)
- net M3_ONOFF: now reaches U1.62 (NCSI0-D11)
- net M3_ONOFF: now also X4.1 (Pin_1)
- removed net VCC: C5.1, C7.1, U2.2 (VIN), X1.1 (Pin_1), X2.1 (Pin_1), X3.1 (Pin_1), X4.1 (Pin_1)
- new net: C5.1, C7.1, D1.1 (+), D2.1 (K), U2.2 (VIN), X5.1 (Pin_1)
- new net: C10.2, R13.2, R14.2
- new net: R24.1, X7.10
- new net: R13.1, T1.15 (C_TX)
- new net: R23.1, X7.12
- new net: R14.1, T1.10 (C_RX)
- new net TO0_N: T1.14 (TX-), X7.2
- new net TO0_P: T1.16 (TX+), X7.1
- new net TO1_N: T1.9 (RX-), X7.6
- new net TO1_P: T1.11 (RX+), X7.3
- new net VIN1: D1.3, X7.4, X7.5
- new net VIN2: D1.4, X7.7, X7.8
- no-connect marks 153 -> 148

Commit message: routing procs
Parts:
- removed H6: M3, MountingHole:MountingHole_3.5mm_Pad, symbol Mechanical:MountingHole_Pad
- X1, X2, X3, X4: value S4B-XH -> B4B-XH; footprint Connector_JST:JST_XH_S4B-XH-A_1x04_P2.50mm_Horizontal -> Connector_JST:JST_XH_B4B-XH-A_1x04_P2.50mm_Vertical
Changed lines of the file:
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@@
   (junction (at 198.12 269.24) (diameter 0) (color 0 0 0 0)
   )
-  (junction (at 208.28 269.24) (diameter 0) (color 0 0 0 0)
-  )
   (junction (at 120.65 163.83) (diameter 0) (color 0 0 0 0)
   )
@@
     (stroke (width 0) (type default) (color 0 0 0 0))
   )
-  (wire (pts (xy 203.2 269.24) (xy 208.28 269.24))
-    (stroke (width 0) (type default) (color 0 0 0 0))
-  )
   (wire (pts (xy 166.37 227.33) (xy 166.37 229.87))
     (stroke (width 0) (type default) (color 0 0 0 0))
@@
       (effects (font (size 1.27 1.27)) (justify left))
     )
-    (property "Value" "S4B-XH" (id 1) (at 97.282 245.5422 0)
+    (property "Value" "B4B-XH" (id 1) (at 97.282 245.5422 0)
       (effects (font (size 1.27 1.27)) (justify left))
     )
-    (property "Footprint" "Connector_JST:JST_XH_S4B-XH-A_1x04_P2.50mm_Horizontal" (id 2) (at 95.25 242.57 0)
+    (property "Footprint" "Connector_JST:JST_XH_B4B-XH-A_1x04_P2.50mm_Vertical" (id 2) (at 95.25 242.57 0)
       (effects (font (size 1.27 1.27)) hide)
     )
@@
     (pin "1")
   )
-  (symbol (lib_id "Mechanical:MountingHole_Pad") (at 208.28 266.7 0) (unit 1)
-    (in_bom yes) (on_board yes)
-    (property "Reference" "H6" (id 0) (at 207.01 259.08 0)
-      (effects (font (size 1.27 1.27)) (justify left))
-    )
-    (property "Value" "M3" (id 1) (at 207.01 261.62 0)
-      (effects (font (size 1.27 1.27)) (justify left))
-    )
-    (property "Footprint" "MountingHole:MountingHole_3.5mm_Pad" (id 2) (at 208.28 266.7 0)
-      (effects (font (size 1.27 1.27)) hide)
-    )
-    (property "Datasheet" "~" (id 3) (at 208.28 266.7 0)
-      (effects (font (size 1.27 1.27)) hide)
-    )
-    (pin "1")
-  )
   (symbol (lib_id "Connector_Generic:Conn_01x04") (at 95.25 223.52 0) (unit 1)
     (in_bom yes) (on_board yes) (fields_autoplaced)
@@
       (effects (font (size 1.27 1.27)) (justify left))
     )
-    (property "Value" "S4B-XH" (id 1) (at 97.282 226.4922 0)
+    (property "Value" "B4B-XH" (id 1) (at 97.282 226.4922 0)
       (effects (font (size 1.27 1.27)) (justify left))
     )
-    (property "Footprint" "Connector_JST:JST_XH_S4B-XH-A_1x04_P2.50mm_Horizontal" (id 2) (at 95.25 223.52 0)
+    (property "Footprint" "Connector_JST:JST_XH_B4B-XH-A_1x04_P2.50mm_Vertical" (id 2) (at 95.25 223.52 0)
       (effects (font (size 1.27 1.27)) hide)
     )
@@
       (effects (font (size 1.27 1.27)) (justify left))
     )
-    (property "Value" "S4B-XH" (id 1) (at 97.282 264.5922 0)
+    (property "Value" "B4B-XH" (id 1) (at 97.282 264.5922 0)
       (effects (font (size 1.27 1.27)) (justify left))
     )
-    (property "Footprint" "Connector_JST:JST_XH_S4B-XH-A_1x04_P2.50mm_Horizontal" (id 2) (at 95.25 261.62 0)
+    (property "Footprint" "Connector_JST:JST_XH_B4B-XH-A_1x04_P2.50mm_Vertical" (id 2) (at 95.25 261.62 0)
       (effects (font (size 1.27 1.27)) hide)
     )
@@
     (pin "4")
   )
-  (symbol (lib_id "power:GND") (at 208.28 269.24 0) (unit 1)
+  (symbol (lib_id "power:GND") (at 203.2 269.24 0) (unit 1)
     (in_bom yes) (on_board yes)
-    (property "Reference" "#PWR050" (id 0) (at 208.28 275.59 0)
+    (property "Reference" "#PWR050" (id 0) (at 203.2 275.59 0)
       (effects (font (size 1.27 1.27)) hide)
     )
-    (property "Value" "GND" (id 1) (at 208.28 273.05 0))
-    (property "Footprint" "" (id 2) (at 208.28 269.24 0)
+    (property "Value" "GND" (id 1) (at 203.2 273.05 0))
+    (property "Footprint" "" (id 2) (at 203.2 269.24 0)
       (effects (font (size 1.27 1.27)) hide)
     )
-    (property "Datasheet" "" (id 3) (at 208.28 269.24 0)
+    (property "Datasheet" "" (id 3) (at 203.2 269.24 0)
       (effects (font (size 1.27 1.27)) hide)
     )
@@
       (effects (font (size 1.27 1.27)) (justify left))
     )
-    (property "Value" "S4B-XH" (id 1) (at 97.282 282.3722 0)
+    (property "Value" "B4B-XH" (id 1) (at 97.282 282.3722 0)
       (effects (font (size 1.27 1.27)) (justify left))
     )
-    (property "Footprint" "Connector_JST:JST_XH_S4B-XH-A_1x04_P2.50mm_Horizontal" (id 2) (at 95.25 279.4 0)
+    (property "Footprint" "Connector_JST:JST_XH_B4B-XH-A_1x04_P2.50mm_Vertical" (id 2) (at 95.25 279.4 0)
       (effects (font (size 1.27 1.27)) hide)
     )
@@
       (reference "H5") (unit 1) (value "M3") (footprint "MountingHole:MountingHole_3.5mm_Pad")
     )
-    (path "/db4e52e1-96d1-4aa6-a348-80003a63750a"
-      (reference "H6") (unit 1) (value "M3") (footprint "MountingHole:MountingHole_3.5mm_Pad")
-    )
     (path "/1e513890-8543-40da-acda-0dd52e2841ee"
       (reference "J1") (unit 1) (value "Header") (footprint "Connector_PinHeader_2.54mm:PinHeader_1x03_P2.54mm_Vertical")
@@
     )
     (path "/db9414fa-063a-4929-bf05-37dc6e41cabd"
-      (reference "X1") (unit 1) (value "S4B-XH") (footprint "Connector_JST:JST_XH_S4B-XH-A_1x04_P2.50mm_Horizontal")
+      (reference "X1") (unit 1) (value "B4B-XH") (footprint "Connector_JST:JST_XH_B4B-XH-A_1x04_P2.50mm_Vertical")
     )
     (path "/90c0b5a3-65e7-4730-9ce6-fa4b9000de01"
-      (reference "X2") (unit 1) (value "S4B-XH") (footprint "Connector_JST:JST_XH_S4B-XH-A_1x04_P2.50mm_Horizontal")
+      (reference "X2") (unit 1) (value "B4B-XH") (footprint "Connector_JST:JST_XH_B4B-XH-A_1x04_P2.50mm_Vertical")
     )
     (path "/e0f58b1f-6ecc-44e5-9b03-ae9ec1369882"
-      (reference "X3") (unit 1) (value "S4B-XH") (footprint "Connector_JST:JST_XH_S4B-XH-A_1x04_P2.50mm_Horizontal")
+      (reference "X3") (unit 1) (value "B4B-XH") (footprint "Connector_JST:JST_XH_B4B-XH-A_1x04_P2.50mm_Vertical")
     )
     (path "/fd600413-06c6-4205-8b40-acf6eebb9eeb"
-      (reference "X4") (unit 1) (value "S4B-XH") (footprint "Connector_JST:JST_XH_S4B-XH-A_1x04_P2.50mm_Horizontal")
+      (reference "X4") (unit 1) (value "B4B-XH") (footprint "Connector_JST:JST_XH_B4B-XH-A_1x04_P2.50mm_Vertical")
     )
     (path "/8b9396b8-b6ea-428c-8883-bab5709183be"

Commit message: Modems board ready
Parts:
- added C23: 100u 50V, Capacitor_SMD:CP_Elec_10x10.5, symbol Device:C_Polarized
Connections:
- net GND: now also C23.2
- net at C5.1, C7.1, D1.1 (+)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: now also C23.1
Other:
- moved on the sheet: D2, D3, J1, R2, R3, R4, X5

Commit message: mcu_pdb_routing
Connections:
- net M0_ONOFF: now also U1.17 (LVDS1-D3P); no longer U1.58 (NCSI0-D14)
- net M1_ONOFF: now also U1.16 (LVDS1-D3N); no longer U1.59 (NCSI0-D13)
- net M2_ONOFF: now also U1.14 (LVDS1-D1N); no longer U1.61 (NCSI0-D12)
- net M3_ONOFF: now also U1.13 (LVDS1-D1P); no longer U1.62 (NCSI0-D11)
- net STAT_LED: now also U1.L2 (UART5-RX); no longer U1.56 (NCSI0-D15)
- net UART0_RX: now also R3.2; no longer R4.2
- net UART0_TX: now also R4.2; no longer R3.2
Changed lines of the file:
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@@
   (no_connect (at 73.66 157.48))
   (no_connect (at 40.64 86.36))
+  (no_connect (at 40.64 165.1))
   (no_connect (at 40.64 38.1))
   (no_connect (at 73.66 261.62))
@@
   (no_connect (at 73.66 101.6))
   (no_connect (at 40.64 134.62))
-  (no_connect (at 40.64 48.26))
   (no_connect (at 73.66 88.9))
+  (no_connect (at 40.64 172.72))
   (no_connect (at 40.64 271.78))
   (no_connect (at 40.64 251.46))
@@
   (no_connect (at 40.64 294.64))
   (no_connect (at 40.64 279.4))
-  (no_connect (at 40.64 231.14))
   (no_connect (at 73.66 256.54))
   (no_connect (at 40.64 284.48))
@@
   (no_connect (at 73.66 274.32))
   (no_connect (at 40.64 147.32))
+  (no_connect (at 40.64 157.48))
   (no_connect (at 73.66 170.18))
   (no_connect (at 40.64 220.98))
@@
   (no_connect (at 73.66 292.1))
   (no_connect (at 40.64 193.04))
+  (no_connect (at 40.64 170.18))
   (no_connect (at 73.66 137.16))
-  (no_connect (at 40.64 50.8))
   (no_connect (at 40.64 187.96))
   (no_connect (at 73.66 238.76))
@@
   (no_connect (at 40.64 246.38))
   (no_connect (at 73.66 236.22))
-  (no_connect (at 40.64 55.88))
   (no_connect (at 73.66 78.74))
   (no_connect (at 73.66 93.98))
+  (no_connect (at 40.64 162.56))
   (no_connect (at 73.66 279.4))
   (no_connect (at 40.64 261.62))
@@
   (no_connect (at 73.66 116.84))
   (no_connect (at 40.64 289.56))
-  (no_connect (at 40.64 58.42))
   (no_connect (at 40.64 223.52))
   (no_connect (at 40.64 154.94))
@@
     (stroke (width 0) (type default) (color 0 0 0 0))
   )
+  (wire (pts (xy 27.94 48.26) (xy 40.64 48.26))
+    (stroke (width 0) (type default) (color 0 0 0 0))
+  )
   (wire (pts (xy 193.04 269.24) (xy 198.12 269.24))
     (stroke (width 0) (type default) (color 0 0 0 0))
@@
     (stroke (width 0) (type default) (color 0 0 0 0))
   )
-  (wire (pts (xy 29.21 165.1) (xy 40.64 165.1))
-    (stroke (width 0) (type default) (color 0 0 0 0))
-  )
   (wire (pts (xy 120.65 128.27) (xy 128.27 128.27))
     (stroke (width 0) (type default) (color 0 0 0 0))
@@
     (stroke (width 0) (type default) (color 0 0 0 0))
   )
+  (wire (pts (xy 27.94 50.8) (xy 40.64 50.8))
+    (stroke (width 0) (type default) (color 0 0 0 0))
+  )
   (wire (pts (xy 191.77 139.7) (xy 191.77 148.59))
     (stroke (width 0) (type default) (color 0 0 0 0))
@@
     (stroke (width 0) (type default) (color 0 0 0 0))
   )
+  (wire (pts (xy 27.94 55.88) (xy 40.64 55.88))
+    (stroke (width 0) (type default) (color 0 0 0 0))
+  )
   (wire (pts (xy 74.93 60.96) (xy 74.93 53.34))
     (stroke (width 0) (type default) (color 0 0 0 0))
@@
     (stroke (width 0) (type default) (color 0 0 0 0))
   )
-  (wire (pts (xy 29.21 157.48) (xy 40.64 157.48))
-    (stroke (width 0) (type default) (color 0 0 0 0))
-  )
   (wire (pts (xy 39.37 91.44) (xy 39.37 99.06))
     (stroke (width 0) (type default) (color 0 0 0 0))
@@
     (stroke (width 0) (type default) (color 0 0 0 0))
   )
+  (wire (pts (xy 27.94 58.42) (xy 40.64 58.42))
+    (stroke (width 0) (type default) (color 0 0 0 0))
+  )
   (wire (pts (xy 133.35 30.48) (xy 133.35 31.75))
     (stroke (width 0) (type default) (color 0 0 0 0))
   )
-  (wire (pts (xy 29.21 170.18) (xy 40.64 170.18))
-    (stroke (width 0) (type default) (color 0 0 0 0))
-  )
   (wire (pts (xy 39.37 60.96) (xy 39.37 68.58))
     (stroke (width 0) (type default) (color 0 0 0 0))
@@
     (stroke (width 0) (type default) (color 0 0 0 0))
   )
-  (wire (pts (xy 29.21 172.72) (xy 40.64 172.72))
-    (stroke (width 0) (type default) (color 0 0 0 0))
-  )
   (wire (pts (xy 105.41 158.75) (xy 132.08 158.75))
     (stroke (width 0) (type default) (color 0 0 0 0))
@@
     (stroke (width 0) (type default) (color 0 0 0 0))
   )
-  (wire (pts (xy 29.21 162.56) (xy 40.64 162.56))
-    (stroke (width 0) (type default) (color 0 0 0 0))
-  )
   (wire (pts (xy 172.72 30.48) (xy 172.72 40.64))
     (stroke (width 0) (type default) (color 0 0 0 0))
@@
     (stroke (width 0) (type default) (color 0 0 0 0))
   )
+  (wire (pts (xy 29.21 231.14) (xy 40.64 231.14))
+    (stroke (width 0) (type default) (color 0 0 0 0))
+  )
   (wire (pts (xy 182.88 110.49) (xy 191.77 110.49))
     (stroke (width 0) (type default) (color 0 0 0 0))
@@
     (effects (font (size 1.27 1.27)) (justify left bottom))
   )
-  (label "M0_ONOFF" (at 29.21 162.56 0)
+  (label "M0_ONOFF" (at 27.94 58.42 0)
     (effects (font (size 1.27 1.27)) (justify left bottom))
   )
@@
     (effects (font (size 1.27 1.27)) (justify left bottom))
   )
-  (label "UART0_TX" (at 95.25 78.74 0)
-    (effects (font (size 1.27 1.27)) (justify left bottom))
-  )
-  (label "M1_ONOFF" (at 29.21 165.1 0)
+  (label "UART0_TX" (at 95.25 81.28 0)
+    (effects (font (size 1.27 1.27)) (justify left bottom))
+  )
+  (label "M1_ONOFF" (at 27.94 55.88 0)
     (effects (font (size 1.27 1.27)) (justify left bottom))
   )
@@
     (effects (font (size 1.27 1.27)) (justify right bottom))
   )
-  (label "M2_ONOFF" (at 29.21 170.18 0)
+  (label "M2_ONOFF" (at 27.94 50.8 0)
     (effects (font (size 1.27 1.27)) (justify left bottom))
   )
@@
     (effects (font (size 1.27 1.27)) (justify left bottom))
   )
-  (label "UART0_RX" (at 95.25 81.28 0)
+  (label "UART0_RX" (at 95.25 78.74 0)
     (effects (font (size 1.27 1.27)) (justify left bottom))
   )
@@
     (effects (font (size 1.27 1.27)) (justify right bottom))
   )
-  (label "STAT_LED" (at 29.21 157.48 0)
+  (label "STAT_LED" (at 29.21 231.14 0)
     (effects (font (size 1.27 1.27)) (justify left bottom))
   )
@@
     (effects (font (size 1.27 1.27)) (justify left bottom))
   )
-  (label "M3_ONOFF" (at 29.21 172.72 0)
-    (effects (font (size 1.27 1.27)) (justify left bottom))
-  )
+  (label "M3_ONOFF" (at 27.94 48.26 0)
+    (effects (font (size 1.27 1.27)) (justify left bottom))
+  )

Commit message: Ready for order
Parts:
- R13, R14: value 75 -> 75R
- U2: value TPS54540 -> TPS54340
Changed lines of the file:
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@@
       (effects (font (size 1.27 1.27)) (justify left))
     )
-    (property "Value" "75" (id 1) (at 144.78 234.95 0)
+    (property "Value" "75R" (id 1) (at 143.51 234.95 0)
       (effects (font (size 1.27 1.27)) (justify left))
     )
@@
       (effects (font (size 1.27 1.27)) (justify left))
     )
-    (property "Value" "75" (id 1) (at 157.48 234.95 0)
+    (property "Value" "75R" (id 1) (at 157.48 234.95 0)
       (effects (font (size 1.27 1.27)) (justify left))
     )
@@
     (in_bom yes) (on_board yes) (fields_autoplaced)
     (property "Reference" "U2" (id 0) (at 149.86 19.1602 0))
-    (property "Value" "TPS54540" (id 1) (at 149.86 21.6971 0))
+    (property "Value" "TPS54340" (id 1) (at 149.86 21.6971 0))
     (property "Footprint" "Package_SO:TI_SO-PowerPAD-8_ThermalVias" (id 2) (at 151.13 41.91 0)
       (effects (font (size 1.27 1.27) italic) (justify left) hide)
@@
     )
     (path "/24554a85-f657-4786-9b7a-58f33b046888"
-      (reference "R13") (unit 1) (value "75") (footprint "Resistor_SMD:R_0603_1608Metric")
+      (reference "R13") (unit 1) (value "75R") (footprint "Resistor_SMD:R_0603_1608Metric")
     )
     (path "/50e354ff-4c20-4cd3-853a-81a8dac19294"
-      (reference "R14") (unit 1) (value "75") (footprint "Resistor_SMD:R_0603_1608Metric")
+      (reference "R14") (unit 1) (value "75R") (footprint "Resistor_SMD:R_0603_1608Metric")
     )
     (path "/513b4f1c-29e0-4352-a51c-dd39a0fd8c58"
@@
     )
     (path "/d711834b-28ef-4737-b3c4-a70e3e15207a"
-      (reference "U2") (unit 1) (value "TPS54540") (footprint "Package_SO:TI_SO-PowerPAD-8_ThermalVias")
+      (reference "U2") (unit 1) (value "TPS54340") (footprint "Package_SO:TI_SO-PowerPAD-8_ThermalVias")
     )
     (path "/441cd409-d7e6-4d66-b6ef-d002740b33e6"
